File: pcb/pcb-01/sch01-input.kicad_sch (KiCad schematic)
At the start: 11 parts, among them Q1 DMP6023LE-13

Commit message: pcb: capture SCH-04..07, full-project ERC clean
Parallel agent capture of the remaining blocks: SCH-04 ESP32-C6 (full GPIO
map, boot straps, USB chain with TPD2EUSB30 on the connector side of the
22R), SCH-05 permission + watchdog (both '1G74s with the review-fixed /PRE
topologies, six-BAT54H wired-OR, TPS3435 pinout C, separate 100R heartbeat
feeds), SCH-06 analog tach (TPS7A16 protected rail with 10 nF DELAY, LM2907
with grounded CP1 and emitter load, TLV1701 trip stage with C2 DNP ladder),
SCH-07 connectors J1-J8 + 28 test points + DNP input-fuse footprint.

ERC: 0 errors after PWR_FLAGs on VM24/AGND/PGND/TACH_LDO_IN and demoting
the MCF's duplicate OUTx/VM/PGND pins to passive. Konnect never refreshes a
sheet's embedded lib_symbols copy (delete + re-add reuses the stale def), so
that one fix was a keyword-only text edit of three pin types, verified by
kicad-cli's full parse. Remaining 41 warnings are two benign classes:
local+global same-name labels (our labeling convention) and embedded-vs-
library symbol formatting drift.

Vendored Konnect agents re-pinned from dead claude-sonnet-4-20250514 to
claude-sonnet-5.
Changed lines of the file:
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@@
+      (justify left bottom))
+)
+  (label "VM24"
+    (at 219.71 71.12 0)
+    (effects
+      (font
+        (size 1.27 1.27))
+      (justify left bottom))
+)
+  (label "PGND"
+    (at 219.71 78.74 0)
+    (effects
+      (font
+        (size 1.27 1.27))
+      (justify left bottom))
+)
+  (label "VM24"
+    (at 69.85 95.25 0)
+    (effects
+      (font
+        (size 1.27 1.27))
+      (justify left bottom))
+)
+  (label "PGND"
+    (at 80.01 95.25 0)
+    (effects
+      (font
+        (size 1.27 1.27))
+      (justify left bottom))
+)
+  (label "AGND"
+    (at 90.17 95.25 0)
+    (effects
+      (font
+        (size 1.27 1.27))
       (justify left bottom))
 )
@@
         (font
           (size 1.27 1.27))))
-        (property "DNP" "DNP"
-      (at 0 0 0)
-      (effects (font (size 1.27 1.27)) (hide yes))
-    )
+    (property "DNP" "DNP"
+      (at 0 0 0)
+      (effects
+        (font
+          (size 1.27 1.27))
+        (hide yes)))
     (instances
       (project "sch01-input"
@@
           (reference "C6")
           (unit 1)))))
-  (label "VM24"
-    (at 219.71 71.12 0)
-    (fields_autoplaced yes)
-    (effects (font (size 1.27 1.27)) (justify left bottom))
-  )
-  (label "PGND"
-    (at 219.71 78.74000000000001 0)
-    (fields_autoplaced yes)
-    (effects (font (size 1.27 1.27)) (justify left bottom))
-  ))
+  (symbol
+    (lib_id "power:PWR_FLAG")
+    (at 69.85 95.25 0)
+    (unit 1)
+    (in_bom yes)
+    (on_board yes)
+    (dnp no)
+    (property "Reference" "#FLG01"
+      (at 69.85 91.44 0)
+      (hide yes)
+      (effects
+        (font
+          (size 1.27 1.27))))
+    (property "Value" "PWR_FLAG"
+      (at 69.85 99.06 0)
+      (effects
+        (font
+          (size 1.27 1.27))))
+    (property "Footprint" ""
+      (at 69.85 95.25 0)
+      (hide yes)
+      (effects
+        (font
+          (size 1.27 1.27))))
+    (property "Datasheet" ""
+      (at 69.85 95.25 0)
+      (hide yes)
+      (effects
+        (font
+          (size 1.27 1.27))))
+    (instances
+      (project "sch01-input"
+        (path "/f4787083-75cc-4a54-9808-7f276fa01d58"
+          (reference "?")
+          (unit 1)))))
+  (symbol
+    (lib_id "power:PWR_FLAG")
+    (at 80.01 95.25 0)
+    (unit 1)
+    (in_bom yes)
+    (on_board yes)
+    (dnp no)
+    (property "Reference" "#FLG02"
+      (at 80.01 91.44 0)
+      (hide yes)
+      (effects
+        (font
+          (size 1.27 1.27))))
+    (property "Value" "PWR_FLAG"
+      (at 80.01 99.06 0)
+      (effects
+        (font
+          (size 1.27 1.27))))
+    (property "Footprint" ""
+      (at 80.01 95.25 0)
+      (hide yes)
+      (effects
+        (font
+          (size 1.27 1.27))))
+    (property "Datasheet" ""
+      (at 80.01 95.25 0)
+      (hide yes)
+      (effects
+        (font
+          (size 1.27 1.27))))
+    (instances
+      (project "sch01-input"
+        (path "/f4787083-75cc-4a54-9808-7f276fa01d58"
+          (reference "?")
+          (unit 1)))))
+  (symbol
+    (lib_id "power:PWR_FLAG")
+    (at 90.17 95.25 0)
+    (unit 1)
+    (in_bom yes)
+    (on_board yes)
+    (dnp no)
+    (property "Reference" "#FLG03"
+      (at 90.17 91.44 0)
+      (hide yes)
+      (effects
+        (font
+          (size 1.27 1.27))))
+    (property "Value" "PWR_FLAG"
+      (at 90.17 99.06 0)
+      (effects
+        (font
+          (size 1.27 1.27))))
+    (property "Footprint" ""
+      (at 90.17 95.25 0)
+      (hide yes)
+      (effects
+        (font
+          (size 1.27 1.27))))
+    (property "Datasheet" ""
+      (at 90.17 95.25 0)
+      (hide yes)
+      (effects
+        (font
+          (size 1.27 1.27))))
+    (instances
+      (project "sch01-input"
+        (path "/f4787083-75cc-4a54-9808-7f276fa01d58"
+          (reference "?")
+          (unit 1)))))
+)
