File: pcb/pcb-01/sch06-tach.kicad_sch (KiCad schematic)
At the start: 0 parts

Commit message: pcb: capture SCH-04..07, full-project ERC clean
Parallel agent capture of the remaining blocks: SCH-04 ESP32-C6 (full GPIO
map, boot straps, USB chain with TPD2EUSB30 on the connector side of the
22R), SCH-05 permission + watchdog (both '1G74s with the review-fixed /PRE
topologies, six-BAT54H wired-OR, TPS3435 pinout C, separate 100R heartbeat
feeds), SCH-06 analog tach (TPS7A16 protected rail with 10 nF DELAY, LM2907
with grounded CP1 and emitter load, TLV1701 trip stage with C2 DNP ladder),
SCH-07 connectors J1-J8 + 28 test points + DNP input-fuse footprint.

ERC: 0 errors after PWR_FLAGs on VM24/AGND/PGND/TACH_LDO_IN and demoting
the MCF's duplicate OUTx/VM/PGND pins to passive. Konnect never refreshes a
sheet's embedded lib_symbols copy (delete + re-add reuses the stale def), so
that one fix was a keyword-only text edit of three pin types, verified by
kicad-cli's full parse. Remaining 41 warnings are two benign classes:
local+global same-name labels (our labeling convention) and embedded-vs-
library symbol formatting drift.

Vendored Konnect agents re-pinned from dead claude-sonnet-4-20250514 to
claude-sonnet-5.
Parts:
- added C26: 10uF 63V, Capacitor_SMD:C_1210_3225Metric, symbol Device:C
- added C27: 100nF 100V, Capacitor_SMD:C_0805_2012Metric, symbol Device:C
- added C28: 10uF 25V, Capacitor_SMD:C_1210_3225Metric, symbol Device:C
- added C29, C33: 100nF, Capacitor_SMD:C_0603_1608Metric, symbol Device:C
- added C30: 10nF 50V C0G, Capacitor_SMD:C_0603_1608Metric, symbol Device:C
- added C31: 10nF, Capacitor_SMD:C_0402_1005Metric, symbol Device:C
- added C32: 1nF C0G, Capacitor_SMD:C_0402_1005Metric, symbol Device:C
- added C34: 100nF 1% C0G, Capacitor_SMD:C_0603_1608Metric, symbol Device:C
- added C35: 2.2uF 16V X7R, Capacitor_SMD:C_0805_2012Metric, symbol Device:C
- added C36: 470nF, Capacitor_SMD:C_0805_2012Metric, symbol Device:C
- added C37: 1uF, Capacitor_SMD:C_0805_2012Metric, symbol Device:C
- added C38: 3.3uF, Capacitor_SMD:C_0805_2012Metric, symbol Device:C
- added C39: 4.7uF, Capacitor_SMD:C_0805_2012Metric, symbol Device:C
- added C40: 6.8uF, Capacitor_SMD:C_0805_2012Metric, symbol Device:C
- added C41: 100nF, Capacitor_SMD:C_0402_1005Metric, symbol Device:C
- added D9: BAT54S, Package_TO_SOT_SMD:SOT-23, symbol Diode:BAT54S
- added Q3: 2N7002, Package_TO_SOT_SMD:SOT-23, symbol Transistor_FET:2N7002
- added R39: 47R 1W, Resistor_SMD:R_2512_6332Metric, symbol Device:R
- added R40: 910k 0.1%, Resistor_SMD:R_0402_1005Metric, symbol Device:R
- added R41: 100k 0.1%, Resistor_SMD:R_0402_1005Metric, symbol Device:R
- added R42, R44, R46, R47, R49: 10k, Resistor_SMD:R_0402_1005Metric, symbol Device:R
- added R43: 100k, Resistor_SMD:R_0402_1005Metric, symbol Device:R
- added R45: 100R, Resistor_SMD:R_0402_1005Metric, symbol Device:R
- added R48: 562k 0.1%, Resistor_SMD:R_0402_1005Metric, symbol Device:R
- added R50: 10.0k, Resistor_SMD:R_0402_1005Metric, symbol Device:R
- added R51: 47.0k 0.1%, Resistor_SMD:R_0402_1005Metric, symbol Device:R
- added R52: 10.0k 0.1%, Resistor_SMD:R_0402_1005Metric, symbol Device:R
- added R53: 35.7k 0.1%, Resistor_SMD:R_0402_1005Metric, symbol Device:R
- added R54: 90.9k 0.1%, Resistor_SMD:R_0402_1005Metric, symbol Device:R
- added RV1: 200k 10-turn, Potentiometer_SMD:Potentiometer_Bourns_3224W_Vertical, symbol Device:R_Potentiometer_Trim
- added U4: TPS7A1601DGN, Package_SO:MSOP-8-1EP_3x3mm_P0.65mm_EP1.68x1.88mm_ThermalVias, symbol pcb01-parts:TPS7A1601DGN
- added U8: LM2907M-14, Package_SO:SOIC-14_3.9x8.7mm_P1.27mm, symbol pcb01-parts:LM2907M-14
- added U9: TLV1701DBV, Package_TO_SOT_SMD:SOT-23-5, symbol pcb01-parts:TLV1701DBV
Connections:
- new net +12V_TACH: C28.1, C29.1, C30.1, R40.1, R44.1, R46.1, U4.1 (OUT), U8.8 (COL), U8.9 (V+)
- new net 3V3: C41.1, D9.2 (K), R42.1, R50.1, R52.1, U9.5 (V+)
- new net AGND: C26.2, C27.2, C28.2, C29.2, C31.2, C32.2, C33.2, C34.2, C35.2, C36.2, C37.2, C38.2, C39.2, C40.2, C41.2, D9.1 (A), Q3.2 (S), R41.2, R43.2, R47.2, R49.2, R53.2, RV1.2, RV1.3, U4.4 (GND), U4.9 (EP), U8.12 (GND), U9.2 (V-)
- new net HALL_TACH: Q3.1 (G), R43.1
- new net LM_TACHIN: C32.1, R45.2, U8.1 (TACH+)
- new net OVERSPEED_N: R42.2, R50.2, R54.1, U4.3 (PG), U9.4 (OUT)
- new net RSCALE_MID: R48.2, RV1.1
- new net TACH_BIAS: C33.1, R46.2, R47.1, U8.11 (TACH-)
- new net TACH_CP1: C34.1, U8.2 (CP1)
- new net TACH_DELAY: C31.1, U4.7 (DELAY)
- new net TACH_DRAIN: Q3.3 (D), R44.2, R45.1
- new net TACH_FB: C30.2, R40.2, R41.1, U4.2 (FB)
- new net TACH_LDO_IN: C26.1, C27.1, R39.2, U4.5 (EN), U4.8 (IN)
- new net TLV_INN: D9.3 (COM), R51.2, U9.3 (IN-)
- new net VM24: R39.1
- new net VREF: R52.2, R53.1, R54.2, U9.1 (IN+)
- new net VTACH: R49.1, R51.1, U8.10 (IN-), U8.5 (EMIT)
- new net VTACH_RAW: C35.1, C36.1, C37.1, C38.1, C39.1, C40.1, R48.1, U8.3 (CP2), U8.4 (IN+)
- no-connect marks 0 -> 5
Other:
- note added: "PG = TACH_PGOOD_N (wire-OR with comparator output; both open-drain)"
