File: pcb/pcb-01/pcb-01.kicad_sch (KiCad schematic)
At the start: 0 parts

Commit message: pcb: capture SCH-01 input + SCH-02 3V3 rail, custom symbol library
Hierarchical sheets for all seven electrical.md blocks. SCH-01 (reverse PMOS
in the canonical drain-to-RAW24 orientation, zener clamp, TVS, bulk bank +
DNP spare) and SCH-02 (TPSM365R6V3 with EN tied to VM24, BIAS to VOUT, mode
solder jumper defaulted to GND/PFM, PGOOD pull-up) captured and
connection-validated, with MPN/LCSC fields on non-generic parts.

pcb01-parts.kicad_sym carries datasheet-verified symbols for MCF8316D
(D-generation pinout), TPSM365R6V3, TPS7A1601, TLV1701, TPS3435 pinout C,
and LM2907M-14. Konnect's placement path only resolves libraries from the
installed-symbols dir, so the library is symlinked into the KiCad app bundle
(re-create after a KiCad update).
Other:
- added sheet SCH-01 24V Input (sch01-input.kicad_sch)
- added sheet SCH-02 3V3 Rail (sch02-logic-rail.kicad_sch)
- added sheet SCH-03 MCF Power Stage (sch03-mcf-power.kicad_sch)
- added sheet SCH-04 ESP32-C6 Supervisor (sch04-esp32.kicad_sch)
- added sheet SCH-05 Permission + Watchdog (sch05-permission.kicad_sch)
- added sheet SCH-06 Hall Tach (sch06-tach.kicad_sch)
- added sheet SCH-07 Connectors (sch07-connectors.kicad_sch)
Changed lines of the file:
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@@
 (kicad_sch
-	(version 20260306)
-	(generator "eeschema")
-	(generator_version "10.0")
-	(paper "A4")
-	(sheet_instances
-		(path "/"
-			(page "1")
-		)
-	)
-	(embedded_fonts no)
+  (version 20260306)
+  (generator "eeschema")
+  (generator_version "10.0")
+  (paper "A4")
+  (sheet
+    (at 20 30)
+    (size 55 35)
+    (fields_autoplaced)
+    (stroke
+      (width 0.1524)
+      (type solid))
+    (fill
+      (color 0 0 0 0.0))
+    (property "Sheetname" "SCH-01 24V Input"
+      (at 20 29.2 0))
+    (property "Sheetfile" "sch01-input.kicad_sch"
+      (at 20 65.4 0))
+    (instances
+      (project "pcb-01"
+        (path "/d3d2f339-2d54-4348-bfa6-3bbc3f84dd10"
+          (page "2")))))
+  (sheet
+    (at 90 30)
+    (size 55 35)
+    (fields_autoplaced)
+    (stroke
+      (width 0.1524)
+      (type solid))
+    (fill
+      (color 0 0 0 0.0))
+    (property "Sheetname" "SCH-02 3V3 Rail"
+      (at 90 29.2 0))
+    (property "Sheetfile" "sch02-logic-rail.kicad_sch"
+      (at 90 65.4 0))
+    (instances
+      (project "pcb-01"
+        (path "/d3d2f339-2d54-4348-bfa6-3bbc3f84dd10"
+          (page "3")))))
+  (sheet
+    (at 160 30)
+    (size 55 35)
+    (fields_autoplaced)
+    (stroke
+      (width 0.1524)
+      (type solid))
+    (fill
+      (color 0 0 0 0.0))
+    (property "Sheetname" "SCH-03 MCF Power Stage"
+      (at 160 29.2 0))
+    (property "Sheetfile" "sch03-mcf-power.kicad_sch"
+      (at 160 65.4 0))
+    (instances
+      (project "pcb-01"
+        (path "/d3d2f339-2d54-4348-bfa6-3bbc3f84dd10"
+          (page "4")))))
+  (sheet
+    (at 230 30)
+    (size 55 35)
+    (fields_autoplaced)
+    (stroke
+      (width 0.1524)
+      (type solid))
+    (fill
+      (color 0 0 0 0.0))
+    (property "Sheetname" "SCH-04 ESP32-C6 Supervisor"
+      (at 230 29.2 0))
+    (property "Sheetfile" "sch04-esp32.kicad_sch"
+      (at 230 65.4 0))
+    (instances
+      (project "pcb-01"
+        (path "/d3d2f339-2d54-4348-bfa6-3bbc3f84dd10"
+          (page "5")))))
+  (sheet
+    (at 20 110)
+    (size 55 35)
+    (fields_autoplaced)
+    (stroke
+      (width 0.1524)
+      (type solid))
+    (fill
+      (color 0 0 0 0.0))
+    (property "Sheetname" "SCH-05 Permission + Watchdog"
+      (at 20 109.2 0))
+    (property "Sheetfile" "sch05-permission.kicad_sch"
+      (at 20 145.4 0))
+    (instances
+      (project "pcb-01"
+        (path "/d3d2f339-2d54-4348-bfa6-3bbc3f84dd10"
+          (page "6")))))
+  (sheet
+    (at 90 110)
+    (size 55 35)
+    (fields_autoplaced)
+    (stroke
+      (width 0.1524)
+      (type solid))
+    (fill
+      (color 0 0 0 0.0))
+    (property "Sheetname" "SCH-06 Hall Tach"
+      (at 90 109.2 0))
+    (property "Sheetfile" "sch06-tach.kicad_sch"
+      (at 90 145.4 0))
+    (instances
+      (project "pcb-01"
+        (path "/d3d2f339-2d54-4348-bfa6-3bbc3f84dd10"
+          (page "7")))))
+  (sheet
+    (at 160 110)
+    (size 55 35)
+    (fields_autoplaced)
+    (stroke
+      (width 0.1524)
+      (type solid))
+    (fill
+      (color 0 0 0 0.0))
+    (property "Sheetname" "SCH-07 Connectors"
+      (at 160 109.2 0))
+    (property "Sheetfile" "sch07-connectors.kicad_sch"
+      (at 160 145.4 0))
+    (instances
+      (project "pcb-01"
+        (path "/d3d2f339-2d54-4348-bfa6-3bbc3f84dd10"
+          (page "8")))))
+  (embedded_fonts no)
+  (sheet_instances
+    (path "/"
+      (page "1")))
 )
