File: pcb/pcb-01/sch02-logic-rail.kicad_sch (KiCad schematic)
At the start: 8 parts, among them U3 TPSM365R6V3RDNR

Commit message: pcb: custom footprints (MCF RGF, TPSM RDN, TI SM8) + full footprint assignment
pcb01-parts.pretty carries three datasheet-derived footprints: MCF8316D
VQFN-40 RGF0040E (40 pads + 3.7x5.7 EP + 12 POFV thermal vias at 0.3 mm
drill), TI SM8 DCT0008A with TI's 3.8 mm pad-row span (the number KiCad's
generic SSOP-8 gets wrong), and TPSM365R6 RDN0011A. The RDN pattern's
chained dimensions were ambiguous, so pad geometry was pixel-measured from
the 20X/600dpi render of TI drawing 4226623/F and cross-checked against the
direct labels; the VOUT/SW comb pads are simplified to rectangles at the
tooth-tip boundary (noted in the footprint description).

L1 uses KiCad's stock Sunlord SWPA6045S footprint. Every component now has
a footprint; ERC remains 0 errors with only the two known-benign warning
classes.
Parts:
- U3: footprint (none) -> pcb01-parts:TPSM365R6_RDN0011A
Changed lines of the file:
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@@
         (font
           (size 1.27 1.27))))
-    (property "Footprint" ""
+    (property "Footprint" "pcb01-parts:TPSM365R6_RDN0011A"
       (at 110.49 69.85 0)
       (hide yes)

Commit message: pcb: review round 1 fixes — hall pull-up, ground tie, DNP marks, footprints
13-lens board-truth review (netlist as source of truth, spec excluded to
avoid circular validation) found and this commit fixes in the schematic:

- R43 was a 100k pulldown to AGND on HALL_TACH; the DRV5033 is open-drain,
  so the hall line could never go high and the analog overspeed chain could
  never trip. Now 10k pull-up to 3V3 (matching the daughterboard section's
  original intent; the LM2907 spec section contradicted it).
- PGND and AGND had no bridge anywhere (the "wide net tie" was layout-note
  prose only): added NT1 (NetTie-2_SMD_Pad2.0mm) on SCH-03.
- C36-C40 tach filter alternates carried no DNP marking; as captured all six
  caps would be assembled in parallel (~18.5uF, ~12s trip lag). Values now
  say DNP.
- J5 footprint was the vertical BM04B while the BOM ordered the side-entry
  SM04B (mating cable already purchased); footprint corrected.
- U12 TPD2EUSB30 was on SOT-563; the part only exists in DRT 3-pin SOT.
  Now Texas_DRT-3 (stock footprint, cites this exact part).
- R3 PGOOD pull-up moved from VOUT to U3_VCC per TI practice; C17 given a
  rating (22uF 25V X7R).

Spec (docs/electrical.md) updated to match, plus an "Open items from the
2026-07 board-truth review" section for the accepted tradeoffs and firmware
TODOs. bom.csv U12 package corrected. groups.json: C32 reassigned from
dnp_bank to tach (functional filter cap, not an alternate).

ERC: no errors (35 pre-existing same_local_global_label warnings from the
label convention). Board-side sync happens via Update-PCB-from-Schematic.
Connections:
- net 3V3: no longer R3.1
- net U3_VCC: now also R3.1
Changed lines of the file:
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@@
-)
-  (label "3V3"
-    (at 134.62 50.8 0)
-    (effects
-      (font
-        (size 1.27 1.27))
-      (justify left bottom))
 )
   (label "3V3"
@@
     (effects
       (font
+        (size 1.27 1.27))
+      (justify left bottom))
+)
+  (label "U3_VCC"
+    (at 134.62 50.8 0)
+    (effects
+      (font
