File: pcb/pcb-01/sch03-mcf-power.kicad_sch (KiCad schematic)
At the start: 0 parts

Commit message: pcb: capture SCH-03 MCF power stage; buck inductor gate resolved
MCF8316D captured with the D-generation pinout: charge pump, AVDD/DVDD
bypass, aux buck (SW_BK/FB_BK/GND_BK), FG/nFAULT/I2C pull-ups, unused-pin
terminations per the safe-defaults table, NC flags on EXT_CLK and DACOUTs,
phases exported as PHASE_U/V/W.

Buck inductor: SWPA4018S470MT fails the electrical.md Isat >= 910 mA gate
(whole 4018/LPS4018 class is ~0.55 A; LPS5030 doesn't close it either and
no 47 uH XAL40xx exists). Swapped to Sunlord SWPA6045S470MT (1.4 A Isat,
LCSC) with LPS6225-473MRB as the DigiKey alternate; bom.csv and
electrical.md updated together. /pcb skill gains the session's Konnect
quirks (local-only batch labels, field creation, symbol lib resolution,
JLCPCB DB 404, KiCad 10 symbol renames, NC validation, SVG rendering).
Parts:
- added C12: 1uF 16V X7R, Capacitor_SMD:C_0603_1608Metric, symbol Device:C
- added C13: 47nF 100V X7R, Capacitor_SMD:C_0805_2012Metric, symbol Device:C
- added C14: 1uF 10V X7R, Capacitor_SMD:C_0603_1608Metric, symbol Device:C
- added C15: 1uF 6.3V X7R, Capacitor_SMD:C_0603_1608Metric, symbol Device:C
- added C16: 22uF 10V X7R, Capacitor_SMD:C_1210_3225Metric, symbol Device:C
- added L1: 47uH, symbol Device:L
- added R10: 100k, Resistor_SMD:R_0402_1005Metric, symbol Device:R
- added R4, R5, R6, R7: 4.7k, Resistor_SMD:R_0402_1005Metric, symbol Device:R
- added R8, R9: 10k, Resistor_SMD:R_0402_1005Metric, symbol Device:R
- added U1: MCF8316D, symbol pcb01-parts:MCF8316D
Connections:
- new net 3V3: R4.1, R5.1, R6.1, R7.1
- new net AGND: C14.2, C15.2, C16.2, R10.2, R8.2, R9.2, U1.2 (DGND), U1.26 (AGND), U1.4 (GND_BK), U1.41 (EP)
- new net ALARM: U1.39 (ALARM)
- new net BUCK_SW: L1.1, U1.5 (SW_BK)
- new net DIR: R9.1, U1.34 (DIR)
- new net DRVOFF: U1.21 (DRVOFF)
- new net FG: R4.2, U1.29 (FG)
- new net MCF_AVDD: C14.1, U1.27 (AVDD)
- new net MCF_BRAKE: R8.1, U1.35 (BRAKE)
- new net MCF_BUCK: C16.1, L1.2, U1.3 (FB_BK)
- new net MCF_CP: C12.1, U1.8 (CP)
- new net MCF_CPH: C13.1, U1.7 (CPH)
- new net MCF_CPL: C13.2, U1.6 (CPL)
- new net MCF_DVDD: C15.1, U1.1 (DVDD)
- new net MCF_EXT_WD: U1.32 (EXT_WD)
- new net NFAULT: R5.2, U1.40 (nFAULT)
- new net PGND: U1.12 (PGND), U1.15 (PGND), U1.18 (PGND)
- new net PHASE_U: U1.13 (OUTA), U1.14 (OUTA)
- new net PHASE_V: U1.16 (OUTB), U1.17 (OUTB)
- new net PHASE_W: U1.19 (OUTC), U1.20 (OUTC)
- new net SCL: R7.2, U1.31 (SCL)
- new net SDA: R6.2, U1.30 (SDA)
- new net SOX: U1.38 (DACOUT2/SOX)
- new net SPEED: R10.1, U1.28 (SPEED/WAKE)
- new net VM24: C12.2, U1.10 (VM), U1.11 (VM), U1.9 (VM)
- no-connect marks 0 -> 7

Commit message: pcb: capture SCH-04..07, full-project ERC clean
Parallel agent capture of the remaining blocks: SCH-04 ESP32-C6 (full GPIO
map, boot straps, USB chain with TPD2EUSB30 on the connector side of the
22R), SCH-05 permission + watchdog (both '1G74s with the review-fixed /PRE
topologies, six-BAT54H wired-OR, TPS3435 pinout C, separate 100R heartbeat
feeds), SCH-06 analog tach (TPS7A16 protected rail with 10 nF DELAY, LM2907
with grounded CP1 and emitter load, TLV1701 trip stage with C2 DNP ladder),
SCH-07 connectors J1-J8 + 28 test points + DNP input-fuse footprint.

ERC: 0 errors after PWR_FLAGs on VM24/AGND/PGND/TACH_LDO_IN and demoting
the MCF's duplicate OUTx/VM/PGND pins to passive. Konnect never refreshes a
sheet's embedded lib_symbols copy (delete + re-add reuses the stale def), so
that one fix was a keyword-only text edit of three pin types, verified by
kicad-cli's full parse. Remaining 41 warnings are two benign classes:
local+global same-name labels (our labeling convention) and embedded-vs-
library symbol formatting drift.

Vendored Konnect agents re-pinned from dead claude-sonnet-4-20250514 to
claude-sonnet-5.
Parts:
- U1: value MCF8316D -> MCF8316DVRGFR

Commit message: pcb: custom footprints (MCF RGF, TPSM RDN, TI SM8) + full footprint assignment
pcb01-parts.pretty carries three datasheet-derived footprints: MCF8316D
VQFN-40 RGF0040E (40 pads + 3.7x5.7 EP + 12 POFV thermal vias at 0.3 mm
drill), TI SM8 DCT0008A with TI's 3.8 mm pad-row span (the number KiCad's
generic SSOP-8 gets wrong), and TPSM365R6 RDN0011A. The RDN pattern's
chained dimensions were ambiguous, so pad geometry was pixel-measured from
the 20X/600dpi render of TI drawing 4226623/F and cross-checked against the
direct labels; the VOUT/SW comb pads are simplified to rectangles at the
tooth-tip boundary (noted in the footprint description).

L1 uses KiCad's stock Sunlord SWPA6045S footprint. Every component now has
a footprint; ERC remains 0 errors with only the two known-benign warning
classes.
Parts:
- L1: footprint (none) -> Inductor_SMD:L_Sunlord_SWPA6045S
- U1: footprint (none) -> pcb01-parts:MCF8316D_RGF0040E
Changed lines of the file:
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@@
         (font
           (size 1.27 1.27))))
-    (property "Footprint" ""
+    (property "Footprint" "Inductor_SMD:L_Sunlord_SWPA6045S"
       (at 95.25 85.09 0)
       (hide yes)
@@
         (font
           (size 1.27 1.27))))
-    (property "Footprint" ""
+    (property "Footprint" "pcb01-parts:MCF8316D_RGF0040E"
       (at 139.7 90.17 0)
       (hide yes)

Commit message: pcb: review round 1 fixes — hall pull-up, ground tie, DNP marks, footprints
13-lens board-truth review (netlist as source of truth, spec excluded to
avoid circular validation) found and this commit fixes in the schematic:

- R43 was a 100k pulldown to AGND on HALL_TACH; the DRV5033 is open-drain,
  so the hall line could never go high and the analog overspeed chain could
  never trip. Now 10k pull-up to 3V3 (matching the daughterboard section's
  original intent; the LM2907 spec section contradicted it).
- PGND and AGND had no bridge anywhere (the "wide net tie" was layout-note
  prose only): added NT1 (NetTie-2_SMD_Pad2.0mm) on SCH-03.
- C36-C40 tach filter alternates carried no DNP marking; as captured all six
  caps would be assembled in parallel (~18.5uF, ~12s trip lag). Values now
  say DNP.
- J5 footprint was the vertical BM04B while the BOM ordered the side-entry
  SM04B (mating cable already purchased); footprint corrected.
- U12 TPD2EUSB30 was on SOT-563; the part only exists in DRT 3-pin SOT.
  Now Texas_DRT-3 (stock footprint, cites this exact part).
- R3 PGOOD pull-up moved from VOUT to U3_VCC per TI practice; C17 given a
  rating (22uF 25V X7R).

Spec (docs/electrical.md) updated to match, plus an "Open items from the
2026-07 board-truth review" section for the accepted tradeoffs and firmware
TODOs. bom.csv U12 package corrected. groups.json: C32 reassigned from
dnp_bank to tach (functional filter cap, not an alternate).

ERC: no errors (35 pre-existing same_local_global_label warnings from the
label convention). Board-side sync happens via Update-PCB-from-Schematic.
Parts:
- added NT1: PGND-AGND tie, NetTie:NetTie-2_SMD_Pad2.0mm, symbol Device:NetTie_2
Connections:
- net AGND: now also NT1.2
- net PGND: now also NT1.1
Changed lines of the file:
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@@
+      (justify left bottom))
+)
+  (label "PGND"
+    (at 48.26 148.59 0)
+    (effects
+      (font
+        (size 1.27 1.27))
+      (justify left bottom))
+)
+  (label "AGND"
+    (at 53.34 148.59 0)
+    (effects
+      (font
+        (size 1.27 1.27))
       (justify left bottom))
 )
@@
         (font
           (size 1.27 1.27))))
-        (property "MPN" "MCF8316DVRGFR"
+    (property "MPN" "MCF8316DVRGFR"
       (at 0 0 0)
-      (effects (font (size 1.27 1.27)) (hide yes))
-    )
-        (property "LCSC" "C47122159"
+      (effects
+        (font
+          (size 1.27 1.27))
+        (hide yes)))
+    (property "LCSC" "C47122159"
       (at 0 0 0)
-      (effects (font (size 1.27 1.27)) (hide yes))
-    )
+      (effects
+        (font
+          (size 1.27 1.27))
+        (hide yes)))
     (instances
       (project "sch03-mcf-power"
@@
           (reference "U1")
           (unit 1)))))
-)
+  (symbol
+    (lib_id "Device:NetTie_2")
+    (at 50.8 148.59 0)
+    (unit 1)
+    (in_bom yes)
+    (on_board yes)
+    (dnp no)
+    (property "Reference" "NT1"
+      (at 50.8 144.78 0)
+      (effects
+        (font
+          (size 1.27 1.27))))
+    (property "Value" "PGND-AGND tie"
+      (at 50.8 152.4 0)
+      (effects
+        (font
+          (size 1.27 1.27))))
+    (property "Footprint" "NetTie:NetTie-2_SMD_Pad2.0mm"
+      (at 50.8 148.59 0)
+      (hide yes)
+      (effects
+        (font
+          (size 1.27 1.27))))
+    (property "Datasheet" ""
+      (at 50.8 148.59 0)
+      (hide yes)
+      (effects
+        (font
+          (size 1.27 1.27))))
+    (instances
+      (project "sch03-mcf-power"
+        (path "/8fb5e3f8-8338-4744-bcd3-fd635296a010"
+          (reference "NT1")
+          (unit 1)))))
+)
