File: pcb/pcb-01/sch04-esp32.kicad_sch (KiCad schematic)
At the start: 0 parts

Commit message: pcb: capture SCH-04..07, full-project ERC clean
Parallel agent capture of the remaining blocks: SCH-04 ESP32-C6 (full GPIO
map, boot straps, USB chain with TPD2EUSB30 on the connector side of the
22R), SCH-05 permission + watchdog (both '1G74s with the review-fixed /PRE
topologies, six-BAT54H wired-OR, TPS3435 pinout C, separate 100R heartbeat
feeds), SCH-06 analog tach (TPS7A16 protected rail with 10 nF DELAY, LM2907
with grounded CP1 and emitter load, TLV1701 trip stage with C2 DNP ladder),
SCH-07 connectors J1-J8 + 28 test points + DNP input-fuse footprint.

ERC: 0 errors after PWR_FLAGs on VM24/AGND/PGND/TACH_LDO_IN and demoting
the MCF's duplicate OUTx/VM/PGND pins to passive. Konnect never refreshes a
sheet's embedded lib_symbols copy (delete + re-add reuses the stale def), so
that one fix was a keyword-only text edit of three pin types, verified by
kicad-cli's full parse. Remaining 41 warnings are two benign classes:
local+global same-name labels (our labeling convention) and embedded-vs-
library symbol formatting drift.

Vendored Konnect agents re-pinned from dead claude-sonnet-4-20250514 to
claude-sonnet-5.
Parts:
- added C17: 22uF, Capacitor_SMD:C_1210_3225Metric, symbol Device:C
- added C18, C20: 100nF, Capacitor_SMD:C_0402_1005Metric, symbol Device:C
- added C19: 1uF, Capacitor_SMD:C_0402_1005Metric, symbol Device:C
- added R11, R12, R13, R18, R19: 10k, Resistor_SMD:R_0402_1005Metric, symbol Device:R
- added R14, R15: 100R, Resistor_SMD:R_0402_1005Metric, symbol Device:R
- added R16, R17: 0R, Resistor_SMD:R_0402_1005Metric, symbol Device:R
- added R20, R21: 22R, Resistor_SMD:R_0402_1005Metric, symbol Device:R
- added SW1, SW2: SW_Push, Button_Switch_SMD:SW_SPST_PTS645Sx43SMTR92, symbol Switch:SW_Push
- added U12: TPD2EUSB30, Package_TO_SOT_SMD:SOT-563, symbol Power_Protection:TPD2EUSB30
- added U2: ESP32-C6-MINI-1, symbol RF_Module:ESP32-C6-MINI-1
Connections:
- new net 3V3: C17.1, C18.1, R11.1, R12.1, R13.1, R18.1, R19.1, U2.3 (3V3)
- new net AGND: C17.2, C18.2, C19.2, C20.2, SW1.2, SW2.2, U12.3 (GND), U2.1 (GND), U2.11 (GND), U2.14 (GND), U2.2 (GND), U2.36 (GND), U2.37 (GND), U2.38 (GND), U2.39 (GND), U2.40 (GND), U2.41 (GND), U2.42 (GND), U2.43 (GND), U2.44 (GND), U2.45 (GND), U2.46 (GND), U2.47 (GND), U2.48 (GND), U2.49 (GND), U2.50 (GND), U2.51 (GND), U2.52 (GND), U2.53 (GND)
- new net ALARM: U2.19 (IO14)
- new net ARM_PULSE: U2.24 (IO18)
- new net DIR: R15.2
- new net ESP_BOOT: R12.2, SW2.1, U2.23 (IO9)
- new net ESP_DIR: R15.1, U2.6 (IO3)
- new net ESP_EN: C19.1, R11.2, SW1.1, U2.8 (EN)
- new net ESP_GPIO8: R13.2, U2.22 (IO8)
- new net ESP_SCL: R17.1, U2.13 (IO1)
- new net ESP_SDA: R16.1, U2.12 (IO0)
- new net ESP_SPEED: R14.1, U2.5 (IO2)
- new net ESP_USB_DM: R20.1, U2.17 (IO12)
- new net ESP_USB_DP: R21.1, U2.18 (IO13)
- new net FG: U2.26 (IO20)
- new net HALL_TACH: U2.16 (IO7)
- new net MCU_CLEAR_N: R18.2, U2.20 (IO15)
- new net NFAULT: U2.27 (IO21)
- new net PGOOD: U2.28 (IO22)
- new net SCL: R17.2
- new net SDA: R16.2
- new net SPEED: R14.2
- new net TEMP_SENSE: C20.1, R19.2, U2.15 (IO6)
- new net UART_RX: U2.30 (RXD0)
- new net UART_TX: U2.31 (TXD0)
- new net USB_DM: R20.2, U12.2 (D-)
- new net USB_DP: R21.2, U12.1 (D+)
- new net WDO: U2.29 (IO23)
- new net WD_HEARTBEAT: U2.25 (IO19)
- no-connect marks 0 -> 9

Commit message: pcb: custom footprints (MCF RGF, TPSM RDN, TI SM8) + full footprint assignment
pcb01-parts.pretty carries three datasheet-derived footprints: MCF8316D
VQFN-40 RGF0040E (40 pads + 3.7x5.7 EP + 12 POFV thermal vias at 0.3 mm
drill), TI SM8 DCT0008A with TI's 3.8 mm pad-row span (the number KiCad's
generic SSOP-8 gets wrong), and TPSM365R6 RDN0011A. The RDN pattern's
chained dimensions were ambiguous, so pad geometry was pixel-measured from
the 20X/600dpi render of TI drawing 4226623/F and cross-checked against the
direct labels; the VOUT/SW comb pads are simplified to rectangles at the
tooth-tip boundary (noted in the footprint description).

L1 uses KiCad's stock Sunlord SWPA6045S footprint. Every component now has
a footprint; ERC remains 0 errors with only the two known-benign warning
classes.
Parts:
- U2: footprint (none) -> RF_Module:ESP32-C6-MINI-1
Changed lines of the file:
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@@
         (font
           (size 1.27 1.27))))
-    (property "Footprint" ""
+    (property "Footprint" "RF_Module:ESP32-C6-MINI-1"
       (at 139.7 100.33 0)
       (hide yes)

Commit message: pcb: placement toolkit + group briefs; antenna courtyard trimmed to body
pcb/tools/: board_model.py (exact courtyard/pad/net parser incl. fp_circle
radial courtyards and KiCad 10 unnumbered pad nets), apply_positions.py
(bulk file-based position writes with kicad-cli parse verification),
validate_group.py, make_briefs.py, park_unplaced.py, render_board.sh.

U2 now uses pcb01-parts:ESP32-C6-MINI-1_BodyCourtyard - the official
footprint's courtyard covered the whole 32x43mm antenna keepout, banning
parts from the doc's tach zone; the copper keepout zone is retained and
only low-profile parts will enter the band (accepted RF tradeoff). All 147
unpinned parts parked off-board; per-group placement briefs with net
adjacency generated under pcb/pcb-01/placement/.
Parts:
- U2: footprint RF_Module:ESP32-C6-MINI-1 -> pcb01-parts:ESP32-C6-MINI-1_BodyCourtyard
Changed lines of the file:
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@@
         (font
           (size 1.27 1.27))))
-    (property "Footprint" "RF_Module:ESP32-C6-MINI-1"
+    (property "Footprint" "pcb01-parts:ESP32-C6-MINI-1_BodyCourtyard"
       (at 139.7 100.33 0)
       (hide yes)

Commit message: pcb: review round 1 fixes — hall pull-up, ground tie, DNP marks, footprints
13-lens board-truth review (netlist as source of truth, spec excluded to
avoid circular validation) found and this commit fixes in the schematic:

- R43 was a 100k pulldown to AGND on HALL_TACH; the DRV5033 is open-drain,
  so the hall line could never go high and the analog overspeed chain could
  never trip. Now 10k pull-up to 3V3 (matching the daughterboard section's
  original intent; the LM2907 spec section contradicted it).
- PGND and AGND had no bridge anywhere (the "wide net tie" was layout-note
  prose only): added NT1 (NetTie-2_SMD_Pad2.0mm) on SCH-03.
- C36-C40 tach filter alternates carried no DNP marking; as captured all six
  caps would be assembled in parallel (~18.5uF, ~12s trip lag). Values now
  say DNP.
- J5 footprint was the vertical BM04B while the BOM ordered the side-entry
  SM04B (mating cable already purchased); footprint corrected.
- U12 TPD2EUSB30 was on SOT-563; the part only exists in DRT 3-pin SOT.
  Now Texas_DRT-3 (stock footprint, cites this exact part).
- R3 PGOOD pull-up moved from VOUT to U3_VCC per TI practice; C17 given a
  rating (22uF 25V X7R).

Spec (docs/electrical.md) updated to match, plus an "Open items from the
2026-07 board-truth review" section for the accepted tradeoffs and firmware
TODOs. bom.csv U12 package corrected. groups.json: C32 reassigned from
dnp_bank to tach (functional filter cap, not an alternate).

ERC: no errors (35 pre-existing same_local_global_label warnings from the
label convention). Board-side sync happens via Update-PCB-from-Schematic.
Parts:
- C17: value 22uF -> 22uF 25V X7R
- U12: footprint Package_TO_SOT_SMD:SOT-563 -> Package_TO_SOT_SMD:Texas_DRT-3
Changed lines of the file:
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@@
         (font
           (size 1.27 1.27))))
-    (property "Value" "22uF"
+    (property "Value" "22uF 25V X7R"
       (at 100.33 53.34 0)
       (effects
@@
         (font
           (size 1.27 1.27))))
-    (property "Footprint" "Package_TO_SOT_SMD:SOT-563"
+    (property "Footprint" "Package_TO_SOT_SMD:Texas_DRT-3"
       (at 204.47 85.09 0)
       (hide yes)
