File: pcb/pcb-01/pcb-01.kicad_pcb (KiCad board)
At the start: 4 copper layers, 78 x 58 mm, 170 parts, among them J1 POWER, J2 MOTOR, J3 HALL, J4 TEMP, J5 I2C, J6 USB-C, J7 PROGRAM, J8 DNP 2x5 1.27mm, Q1 DMP6023LE-13, Q2 2N7002K, Q3 2N7002, SW1 SW_Push, SW2 SW_Push, SW3 SW_Push, U1 MCF8316DVRGFR, U10 SN74LVC1G17DCKR, U11 SN74LVC1G17DCKR, U12 TPD2EUSB30, U2 ESP32-C6-MINI-1, U3 TPSM365R6V3RDNR, U4 TPS7A1601DGN, U5 SN74LVC1G74DCTR, U6 SN74LVC1G74DCTR, U7 TPS3435CAKAGDD, U8 LM2907M-14, U9 TLV1701DBV

Commit message: pcb: post-routing audit fixes — RAW24 haul widened, SW-node fill keepout
Scripted audits (width-vs-netclass, tach purity, SW-vs-fill, antenna
strip) found two real issues: RAW24's 0.5 mm input haul + undersized
vias (the only Power24 net without a plane), and the AGND B.Cu fill
running 0.30 mm from BUCK_SW for 8 mm. Both fixed and re-verified;
DRC baseline unchanged, zero unconnected.
Routing:
- net RAW24: track 29.9 -> 29.1 mm
Changed lines of the file:
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@@
 	)
 	(segment
-		(start 64.5 79.5)
-		(end 64.5 75.25)
-		(width 0.5)
+		(start 70 73.375)
+		(end 68.225 75.15)
+		(width 2)
 		(layer "F.Cu")
 		(net "RAW24")
 	)
 	(segment
-		(start 70 73.375)
-		(end 68.225 75.15)
+		(start 52.528248 68.471752)
+		(end 55.471752 68.471752)
 		(width 2)
 		(layer "F.Cu")
@@
 	)
 	(segment
-		(start 64.5 81.35)
-		(end 64.6 81.45)
-		(width 0.5)
+		(start 55.471752 68.471752)
+		(end 56.9 69.9)
+		(width 2)
 		(layer "F.Cu")
 		(net "RAW24")
@@
 	(segment
 		(start 52.5 68.5)
-		(end 53.5 68.5)
-		(width 0.5)
+		(end 52.528248 68.471752)
+		(width 2)
 		(layer "F.Cu")
 		(net "RAW24")
@@
 	)
 	(segment
-		(start 64.5 79.5)
-		(end 64.5 81.35)
-		(width 0.5)
-		(layer "F.Cu")
-		(net "RAW24")
-	)
-	(segment
-		(start 64.5 75.25)
+		(start 64.6 81.45)
 		(end 64.6 75.15)
-		(width 0.5)
+		(width 2)
 		(layer "F.Cu")
 		(net "RAW24")
@@
 	)
 	(via
-		(at 53.5 68.5)
-		(size 0.6)
-		(drill 0.3)
+		(at 56.9 69.9)
+		(size 1)
+		(drill 0.5)
 		(layers "F.Cu" "B.Cu")
 		(net "RAW24")
 	)
 	(via
-		(at 64.5 79.5)
-		(size 0.6)
-		(drill 0.3)
+		(at 64.5 77.5)
+		(size 1)
+		(drill 0.5)
 		(layers "F.Cu" "B.Cu")
 		(net "RAW24")
 	)
 	(segment
-		(start 64.5 79.5)
-		(end 53.5 68.5)
-		(width 0.5)
+		(start 56.9 69.9)
+		(end 64.5 77.5)
+		(width 2)
 		(layer "B.Cu")
 		(net "RAW24")
@@
 			)
 		)
+	)
+	(zone
+		(layer "B.Cu")
+		(name "copper-keepout")
+		(hatch edge 0.5)
+		(connect_pads
+			(clearance 0)
+		)
+		(min_thickness 0.25)
+		(keepout
+			(tracks allowed)
+			(vias allowed)
+			(pads allowed)
+			(copperpour not_allowed)
+			(footprints allowed)
+		)
+		(placement
+			(enabled no)
+			(sheetname "")
+		)
+		(fill
+			(thermal_gap 0.5)
+			(thermal_bridge_width 0.5)
+			(island_removal_mode 0)
+		)
+		(polygon
+			(pts
+				(xy 72.9 92.2) (xy 80.2 85.1) (xy 83.2 85.1) (xy 83.3 87.2) (xy 75.4 94.9)
+			)
+		)
