File: pcb/pcb-01-v2/pcb-01-v2.kicad_sch (KiCad schematic)
At the start: 0 parts

Commit message: Build PCB-01 V2 ready-to-route project
Other:
- added sheet SCH-01 24V Input (sch01-input.kicad_sch)
- added sheet SCH-02 3V3 Rail (sch02-logic-rail.kicad_sch)
- added sheet SCH-03 MCF Power Stage (sch03-mcf-power.kicad_sch)
- added sheet SCH-04 Supervisor + Service (sch04-supervisor.kicad_sch)
- added sheet SCH-05 Permission + Watchdog (sch05-permission.kicad_sch)
- added sheet SCH-06 Hall + Overspeed (sch06-overspeed.kicad_sch)
