File: pcb/pcb-01-v2/pcb-01-v2.kicad_pcb (KiCad board)
At the start: 4 copper layers, 88 x 64 mm, 166 parts, among them J1 43045-0200 POWER, J2 43650-0300, J3 B3B-PH-K-S(LF)(SN), J4 USB4105-GF-A, Q1 DMP6023LE-13, Q2 2N7002K-7, Q3 2N7002K-7, SW1 PTS645SK43SMTR92LFS, SW2 PTS645SK43SMTR92LFS, SW3 PTS645SK43SMTR92LFS, U1 MCF8316DVRGFR, U10 SN74LVC1G17DCKR, U11 SN74LVC1G17DCKR, U12 TMP1075DGKR, U13 TPD2EUSB30DRTR, U14 TPD2EUSB30DRTR, U2 ESP32-C6-WROOM-1-N8, U3 TPSM365R6V3RDNR, U4 TPS7A1601ADGNR, U5 SN74LVC1G74DCTR, U6 SN74LVC1G74DCTR, U7 TPS3435CAKAGDDFR, U8 LM2907M-14/NOPB, U9 TLV1701AIDBVR

Commit message: Add U1 VM24 copper landing
Routing:
- net MCF_BUCK: track 0.00 -> 13.5 mm
- net BUCK_SW: track 0.00 -> 10.5 mm
- net MCF_CP: track 0.00 -> 5.89 mm
- net MCF_CPH: track 6.54 -> 1.01 mm, vias 2 -> 1
- net VM24: vias 0 -> 3
- added copper zone on F.Cu, net VM24
Changed lines of the file:
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@@
 		(net "/SCH-04 Supervisor + Service/USB_DP")
+	)
+	(via
+		(at 79.75 95.75)
+		(size 1)
+		(drill 0.5)
+		(layers "F.Cu" "B.Cu")
+		(net "VM24")
+	)
+	(via
+		(at 79.75 97.5)
+		(size 1)
+		(drill 0.5)
+		(layers "F.Cu" "B.Cu")
+		(net "VM24")
+	)
+	(via
+		(at 79.75 99.25)
+		(size 1)
+		(drill 0.5)
+		(layers "F.Cu" "B.Cu")
+		(net "VM24")
 	)
 	(segment
@@
 	)
 	(segment
+		(start 80.908546 95.021002)
+		(end 80.390778 95.021002)
+		(width 0.25)
+		(layer "F.Cu")
+		(net "MCF_CP")
+	)
+	(segment
+		(start 81.179548 94.75)
+		(end 80.908546 95.021002)
+		(width 0.25)
+		(layer "F.Cu")
+		(net "MCF_CP")
+	)
+	(segment
+		(start 80.390778 95.021002)
+		(end 80.024662 94.654886)
+		(width 0.25)
+		(layer "F.Cu")
+		(net "MCF_CP")
+	)
+	(segment
+		(start 79.619843 93.964868)
+		(end 79.619843 93.5)
+		(width 0.25)
+		(layer "F.Cu")
+		(net "MCF_CP")
+	)
+	(segment
+		(start 80.024662 94.654886)
+		(end 80.024662 94.369687)
+		(width 0.25)
+		(layer "F.Cu")
+		(net "MCF_CP")
+	)
+	(segment
+		(start 79.619843 93.5)
+		(end 78.144843 92.025)
+		(width 0.25)
+		(layer "F.Cu")
+		(net "MCF_CP")
+	)
+	(segment
+		(start 80.024662 94.369687)
+		(end 79.619843 93.964868)
+		(width 0.25)
+		(layer "F.Cu")
+		(net "MCF_CP")
+	)
+	(segment
+		(start 81.6 94.75)
+		(end 81.179548 94.75)
+		(width 0.25)
+		(layer "F.Cu")
+		(net "MCF_CP")
+	)
+	(segment
+		(start 78.144843 92.025)
+		(end 77.5 92.025)
+		(width 0.25)
+		(layer "F.Cu")
+		(net "MCF_CP")
+	)
+	(segment
 		(start 88.49 97.5)
 		(end 88.49 94.615)
@@
 	)
 	(segment
-		(start 80.589007 93.472631)
-		(end 80.866376 93.75)
+		(start 73.925 90.425)
+		(end 78.36495 90.425)
+		(width 0.5)
+		(layer "F.Cu")
+		(net "MCF_BUCK")
+	)
+	(segment
+		(start 81.6 92.25)
+		(end 81.073482 92.25)
+		(width 0.25)
+		(layer "F.Cu")
+		(net "MCF_BUCK")
+	)
+	(segment
+		(start 70.35 94)
+		(end 73.925 90.425)
+		(width 0.5)
+		(layer "F.Cu")
+		(net "MCF_BUCK")
+	)
+	(segment
+		(start 78.36495 90.425)
+		(end 80.18995 92.25)
+		(width 0.5)
+		(layer "F.Cu")
+		(net "MCF_BUCK")
+	)
+	(segment
+		(start 80.18995 92.25)
+		(end 81.073482 92.25)
+		(width 0.5)
+		(layer "F.Cu")
+		(net "MCF_BUCK")
+	)
+	(segment
+		(start 78.075 91.125)
+		(end 79.900001 92.95)
+		(width 0.5)
+		(layer "F.Cu")
+		(net "BUCK_SW")
+	)
+	(segment
+		(start 74.85 94)
+		(end 74.85 91.15)
+		(width 0.5)
+		(layer "F.Cu")
+		(net "BUCK_SW")
+	)
+	(segment
+		(start 74.85 91.15)
+		(end 74.875 91.125)
+		(width 0.5)
+		(layer "F.Cu")
+		(net "BUCK_SW")
+	)
+	(segment
+		(start 81.6 93.25)
+		(end 81.073482 93.25)
+		(width 0.25)
+		(layer "F.Cu")
+		(net "BUCK_SW")
+	)
+	(segment
+		(start 80.773482 92.95)
+		(end 80.998482 93.175)
+		(width 0.5)
+		(layer "F.Cu")
+		(net "BUCK_SW")
+	)
+	(segment
+		(start 74.875 91.125)
+		(end 78.075 91.125)
+		(width 0.5)
+		(layer "F.Cu")
+		(net "BUCK_SW")
+	)
+	(segment
+		(start 81.073482 93.25)
+		(end 80.998482 93.175)
+		(width 0.25)
+		(layer "F.Cu")
+		(net "BUCK_SW")
+	)
+	(segment
+		(start 79.900001 92.95)
+		(end 80.773482 92.95)
+		(width 0.5)
+		(layer "F.Cu")
+		(net "BUCK_SW")
+	)
+	(segment
+		(start 80.288859 93.75)
+		(end 80.244843 93.705984)
 		(width 0.25)
 		(layer "F.Cu")
@@
 	)
 	(segment
-		(start 80.866376 93.75)
-		(end 81.6 93.75)
+		(start 81.6 93.75)
+		(end 80.288859 93.75)
 		(width 0.25)
 		(layer "F.Cu")
@@
 	)
 	(via
-		(at 79.15 89.15)
+		(at 79.15 89.25)
 		(size 0.6)
 		(drill 0.3)
@@
 	)
 	(via
-		(at 80.589007 93.472631)
+		(at 80.244843 93.705984)
 		(size 0.6)
 		(drill 0.3)
@@
 	)
 	(segment
-		(start 80.589007 93.472631)
-		(end 80.589007 90.589007)
+		(start 80.244843 90.344843)
+		(end 79.15 89.25)
 		(width 0.25)
 		(layer "B.Cu")
@@
 	)
 	(segment
-		(start 80.589007 90.589007)
-		(end 79.15 89.15)
+		(start 80.244843 93.705984)
+		(end 80.244843 90.344843)
 		(width 0.25)
 		(layer "B.Cu")
@@
 	)
 	(segment
-		(start 80.593946 94.3125)
-		(end 80.656447 94.25)
+		(start 80.795664 94.25)
+		(end 80.649662 94.396002)
 		(width 0.25)
 		(layer "F.Cu")
@@
 	)
 	(segment
-		(start 80.656447 94.25)
-		(end 81.6 94.25)
+		(start 81.6 94.25)
+		(end 80.795664 94.25)
 		(width 0.25)
 		(layer "F.Cu")
@@
 	)
 	(via
-		(at 80.593946 94.3125)
-		(size 0.6)
-		(drill 0.3)
-		(layers "F.Cu" "B.Cu")
-		(net "MCF_CPH")
-	)
-	(via
-		(at 81.05 89.15)
-		(size 0.6)
-		(drill 0.3)
-		(layers "F.Cu" "B.Cu")
-		(net "MCF_CPH")
-	)
-	(segment
-		(start 80.593946 94.3125)
-		(end 80.593947 94.312501)
-		(width 0.25)
-		(layer "B.Cu")
-		(net "MCF_CPH")
-	)
-	(segment
-		(start 80.593947 94.312501)
-		(end 80.633021 94.312501)
-		(width 0.25)
-		(layer "B.Cu")
-		(net "MCF_CPH")
-	)
-	(segment
-		(start 80.633021 94.312501)
-		(end 81.214007 93.731515)
-		(width 0.25)
-		(layer "B.Cu")
-		(net "MCF_CPH")
-	)
-	(segment
-		(start 81.214007 89.314007)
-		(end 81.05 89.15)
-		(width 0.25)
-		(layer "B.Cu")
-		(net "MCF_CPH")
-	)
-	(segment
-		(start 81.214007 93.731515)
-		(end 81.214007 89.314007)
-		(width 0.25)
-		(layer "B.Cu")
+		(at 80.649662 94.396002)
+		(size 0.6)
+		(drill 0.3)
+		(layers "F.Cu" "B.Cu")
 		(net "MCF_CPH")
 	)
@@
 	)
 	(zone
+		(net "VM24")
+		(layer "F.Cu")
+		(name "F.Cu U1 VM24 landing")
+		(hatch edge 0.5)
+		(priority 8)
+		(connect_pads yes
+			(clearance 0.25)
+		)
+		(min_thickness 0.25)
+		(fill yes
+			(thermal_gap 0.5)
+			(thermal_bridge_width 0.5)
+			(island_removal_mode 0)
+		)
+		(polygon
+			(pts
+				(xy 77.25 92.95) (xy 79.1 92.95) (xy 79.1 94.4) (xy 79.45 94.8) (xy 82.05 94.8) (xy 82.05 96.55)
+				(xy 81 96.55) (xy 81 99.7) (xy 78.2 99.7) (xy 78.2 94.25) (xy 77.25 94.05)
+			)
+		)
+	)
+	(zone
